File: keyboard_pcb/keyboard_pcb.kicad_sch (KiCad schematic)
At the start: 0 parts

Commit message: Worked on the project w/ Lapse. Built out concept
Parts:
- added A1: RaspberryPi_Pico, Module:RaspberryPi_Pico_Common_Unspecified, symbol MCU_Module:RaspberryPi_Pico
- added D1: 1N4148, Diode_THT:D_DO-35_SOD27_P7.62mm_Horizontal, symbol Diode:1N4148
- added S1: MX_stab, PCM_marbastlib-mx:STAB_MX_P_6.25u, symbol PCM_marbastlib-mx:MX_stab
- added SW1: SW_Push, symbol Switch:SW_Push
Connections:
- new net: A1.13 (GND), A1.18 (GND), A1.23 (GND), A1.28 (GND), A1.3 (GND), A1.38 (GND), A1.8 (GND)

Commit message: Check journal for more indepth commit
Parts:
- removed A1: RaspberryPi_Pico, Module:RaspberryPi_Pico_Common_Unspecified, symbol MCU_Module:RaspberryPi_Pico
- removed D1: 1N4148, Diode_THT:D_DO-35_SOD27_P7.62mm_Horizontal, symbol Diode:1N4148
- removed SW1: SW_Push, symbol Switch:SW_Push
- added D102, D165, D166, D167, D168, D169, D17, D170, D171, D172, D173, D174, D175, D176, D177, D178, D179, D18, D180, D181, D182, D183, D184, D185, D186, D187, D188, D189, D190, D191, D192, D193, D194, D195, D196, D197, D198, D199, D200, D201, D202, D203, D204, D205, D206, D207, D208, D209, D210, D211, D212, D213, D214, D215, D216, D217, D218, D219, D220, D221, D222, D223, D224, D226, D227, D228, D230, D3, D33, D34, D49, D50, D65, D66, D80, D87, D91, D92, D93, D94, D95: 1N4148, Diode_THT:D_DO-35_SOD27_P7.62mm_Horizontal, symbol Diode:1N4148
- added SW1, SW2, SW4, SW5: RotaryEncoder_Switch_MP, symbol Device:RotaryEncoder_Switch_MP
- added SW102, SW165, SW166, SW167, SW168, SW169, SW17, SW170, SW171, SW172, SW173, SW174, SW175, SW176, SW177, SW178, SW179, SW18, SW180, SW181, SW182, SW183, SW184, SW185, SW186, SW187, SW188, SW189, SW190, SW191, SW192, SW193, SW194, SW195, SW196, SW197, SW198, SW199, SW200, SW201, SW202, SW203, SW204, SW205, SW206, SW207, SW208, SW209, SW210, SW211, SW212, SW213, SW214, SW215, SW216, SW217, SW218, SW219, SW220, SW221, SW222, SW223, SW224, SW226, SW227, SW228, SW230, SW3, SW33, SW34, SW49, SW50, SW65, SW66, SW80, SW87, SW91, SW92, SW93, SW94, SW95: SW_Push, symbol Switch:SW_Push
Connections:
- new net: D177.2 (A), SW177.2
- new net: D165.2 (A), SW165.2
- new net: D170.2 (A), SW170.2
- new net: D91.2 (A), SW91.2
- new net: D198.2 (A), SW198.2
- new net: D223.2 (A), SW223.2
- new net: D181.2 (A), SW181.2
- new net: D227.2 (A), SW227.2
- new net: D175.2 (A), SW175.2
- new net: D102.2 (A), SW102.2
- new net: D217.2 (A), SW217.2
- new net: D174.2 (A), SW174.2
- new net: D168.2 (A), SW168.2
- new net: D219.2 (A), SW219.2
- new net: D197.2 (A), SW197.2
- new net: D80.2 (A), SW80.2
- new net: D33.2 (A), SW33.2
- new net: D213.2 (A), SW213.2
- new net: D171.2 (A), SW171.2
- new net: D92.2 (A), SW92.2
- new net: D183.2 (A), SW183.2
- new net: D211.2 (A), SW211.2
- new net: D184.2 (A), SW184.2
- new net: D166.2 (A), SW166.2
- new net: D200.2 (A), SW200.2
- new net: D180.2 (A), SW180.2
- new net: D212.2 (A), SW212.2
- new net: D209.2 (A), SW209.2
- new net: D182.2 (A), SW182.2
- new net: D214.2 (A), SW214.2
- new net: D3.2 (A), SW3.2
- new net: D93.2 (A), SW93.2
- new net: D187.2 (A), SW187.2
- new net: D167.2 (A), SW167.2
- new net: D169.2 (A), SW169.2
- new net: D226.2 (A), SW226.2
- new net: D216.2 (A), SW216.2
- new net: D173.2 (A), SW173.2
- new net: D222.2 (A), SW222.2
- new net: D178.2 (A), SW178.2
- new net: D205.2 (A), SW205.2
- new net: D204.2 (A), SW204.2
- new net: D18.2 (A), SW18.2
- new net: D207.2 (A), SW207.2
- new net: D228.2 (A), SW228.2
- new net: D87.2 (A), SW87.2
- new net: D201.2 (A), SW201.2
- new net: D186.2 (A), SW186.2
- new net: D17.2 (A), SW17.2
- new net: D94.2 (A), SW94.2
- new net: D221.2 (A), SW221.2
- new net: D218.2 (A), SW218.2
- new net: D206.2 (A), SW206.2
- new net: D190.2 (A), SW190.2
- new net: D220.2 (A), SW220.2
- new net: D50.2 (A), SW50.2
- new net: D224.2 (A), SW224.2
- new net: D202.2 (A), SW202.2
- new net: D196.2 (A), SW196.2
- new net: D195.2 (A), SW195.2
- new net: D189.2 (A), SW189.2
- new net: D230.2 (A), SW230.2
- new net: D191.2 (A), SW191.2
- new net: D179.2 (A), SW179.2
- new net: D185.2 (A), SW185.2
- new net: D192.2 (A), SW192.2
- new net: D95.2 (A), SW95.2
- new net: D34.2 (A), SW34.2
- new net: D208.2 (A), SW208.2
- new net: D215.2 (A), SW215.2
- new net: D188.2 (A), SW188.2
- new net: D176.2 (A), SW176.2
- new net: D194.2 (A), SW194.2
- new net: D172.2 (A), SW172.2
- new net: D210.2 (A), SW210.2
- new net: D193.2 (A), SW193.2
- new net: D65.2 (A), SW65.2
- new net: D203.2 (A), SW203.2
- new net: D66.2 (A), SW66.2
- new net: D199.2 (A), SW199.2
- new net: D49.2 (A), SW49.2
- new net COL0: SW3.1, SW33.1, SW49.1, SW65.1, SW80.1, SW87.1
- new net COL1: SW34.1, SW50.1, SW66.1, SW91.1, SW92.1
- new net COL10: SW201.1, SW202.1, SW203.1, SW204.1, SW205.1, SW206.1
- new net COL11: SW207.1, SW208.1, SW209.1, SW210.1, SW211.1, SW212.1
- new net COL12: SW213.1, SW214.1, SW215.1, SW216.1, SW217.1, SW218.1
- new net COL13: SW219.1, SW220.1, SW221.1, SW222.1, SW223.1, SW224.1
- new net COL14: SW1.S1, SW226.1
- new net COL15: SW227.1, SW228.1
- new net COL16: SW230.1, SW5.S1
- new net COL2: SW102.1, SW165.1, SW17.1, SW93.1, SW94.1, SW95.1
- new net COL3: SW166.1, SW167.1, SW168.1, SW169.1, SW18.1
- new net COL4: SW170.1, SW171.1, SW172.1, SW173.1, SW174.1
- new net COL5: SW175.1, SW176.1, SW177.1, SW178.1, SW179.1
- new net COL6: SW180.1, SW181.1, SW182.1, SW183.1, SW184.1, SW185.1
- new net COL7: SW186.1, SW187.1, SW188.1, SW189.1, SW190.1
- new net COL8: SW191.1, SW192.1, SW193.1, SW194.1, SW195.1
- new net COL9: SW196.1, SW197.1, SW198.1, SW199.1, SW200.1
- new net ROW0: D17.1 (K), D170.1 (K), D175.1 (K), D18.1 (K), D180.1 (K), D186.1 (K), D191.1 (K), D196.1 (K), D201.1 (K), D207.1 (K), D213.1 (K), D219.1 (K), D3.1 (K)
- new net ROW1: D166.1 (K), D171.1 (K), D176.1 (K), D181.1 (K), D187.1 (K), D192.1 (K), D197.1 (K), D202.1 (K), D208.1 (K), D214.1 (K), D220.1 (K), D33.1 (K), D34.1 (K), D93.1 (K)
- new net ROW2: D167.1 (K), D172.1 (K), D177.1 (K), D182.1 (K), D188.1 (K), D193.1 (K), D198.1 (K), D203.1 (K), D209.1 (K), D215.1 (K), D221.1 (K), D49.1 (K), D50.1 (K), D94.1 (K)
- new net ROW3: D168.1 (K), D173.1 (K), D178.1 (K), D183.1 (K), D189.1 (K), D194.1 (K), D199.1 (K), D204.1 (K), D210.1 (K), D216.1 (K), D222.1 (K), D65.1 (K), D66.1 (K), D95.1 (K), SW1.S2, SW5.S2
- new net ROW4: D102.1 (K), D169.1 (K), D174.1 (K), D179.1 (K), D184.1 (K), D190.1 (K), D195.1 (K), D200.1 (K), D205.1 (K), D211.1 (K), D217.1 (K), D223.1 (K), D227.1 (K), D80.1 (K), D91.1 (K)
- new net ROW5: D165.1 (K), D185.1 (K), D206.1 (K), D212.1 (K), D218.1 (K), D224.1 (K), D226.1 (K), D228.1 (K), D230.1 (K), D87.1 (K), D92.1 (K)
Other:
- moved on the sheet: S1
